File: QDevTiny/QDevTiny.kicad_pcb (KiCad board)
At the start: 2 copper layers, 56.1 x 31.8 mm, 31 parts, among them J1 USB_A, J2 Header, J3 ISCP, SW1 RESET_BTN, U1 ATtiny45-20P

Commit message: Update README
Parts:
- removed kibuzzard-63E243CC: G***, kibuzzard-63E243CC
- removed kibuzzard-63E24F9B: G***, kibuzzard-63E24F9B
- removed kibuzzard-63E24FA7: G***, kibuzzard-63E24FA7
- removed kibuzzard-63E24FB3: G***, kibuzzard-63E24FB3
- removed kibuzzard-63E2502C: G***, kibuzzard-63E2502C
- removed kibuzzard-63E25033: G***, kibuzzard-63E25033
- removed kibuzzard-63E25909: G***, kibuzzard-63E25909
- added kibuzzard-63E3F582: G***, kibuzzard-63E3F582, F.Cu at (126.1, 66.0)
- added kibuzzard-63E51F81: G***, kibuzzard-63E51F81, F.Cu at (94.6, 49.5)
- added kibuzzard-63E51F95: G***, kibuzzard-63E51F95, F.Cu at (97.2, 49.4)
- added kibuzzard-63E51F9F: G***, kibuzzard-63E51F9F, F.Cu at (99.7, 49.5)
- added kibuzzard-63E51FA9: G***, kibuzzard-63E51FA9, F.Cu at (102.2, 49.5)
- added kibuzzard-63E51FAF: G***, kibuzzard-63E51FAF, F.Cu at (104.8, 49.5)
- added kibuzzard-63E51FB7: G***, kibuzzard-63E51FB7, F.Cu at (107.3, 50.3)
- C2: footprint Capacitor_THT:C_Disc_D6.0mm_W2.5mm_P5.00mm -> Capacitor_THT:CP_Radial_D4.0mm_P1.50mm
- moved SW1 0.51 mm to (113.6, 51.1)
- moved C2 0.39 mm to (115.7, 46.7)
Routing:
- net PB0: track 73.4 -> 74.6 mm, vias 1 -> 3
- net PB5/R: track 37.4 -> 38.2 mm

Commit message: Start new board and update QDev Tiny README
Parts:
- J3: value ISCP -> ICSP
Changed lines of the file:
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@@
       (effects (font (size 1 1) (thickness 0.15)))
     )
-    (fp_text value "ISCP" (at -2.535 5.065 90) (layer "F.SilkS")
+    (fp_text value "ICSP" (at -2.535 5.065 90) (layer "F.SilkS")
       (effects (font (size 1 1) (thickness 0.15)))
     )
