File: QDevTiny/QDevTiny.kicad_sch (KiCad schematic)
At the start: 17 parts, among them J1 USB_A, J2 Header, J3 ISCP, SW1 RESET_BTN, U1 ATtiny45-20P

Commit message: Update README
Parts:
- C2: footprint Capacitor_THT:C_Disc_D6.0mm_W2.5mm_P5.00mm -> Capacitor_THT:CP_Radial_D4.0mm_P1.50mm
Other:
- note added: "pullup on D- to indicate USB low speed device"
- moved on the sheet: D3
Changed lines of the file:
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@@
   (junction (at 51.435 57.15) (diameter 0) (color 0 0 0 0)
   )
+  (junction (at 159.385 27.305) (diameter 0) (color 0 0 0 0)
+  )
+  (junction (at 29.21 36.195) (diameter 0) (color 0 0 0 0)
+  )
   (junction (at 21.59 52.705) (diameter 0) (color 0 0 0 0)
   )
@@
   )
   (junction (at 99.695 47.625) (diameter 0) (color 0 0 0 0)
+  )
+  (junction (at 159.385 57.785) (diameter 0) (color 0 0 0 0)
   )
   (junction (at 41.275 43.815) (diameter 0) (color 0 0 0 0)
@@
     (stroke (width 0) (type default) (color 0 0 0 0))
   )
+  (wire (pts (xy 159.385 27.305) (xy 168.275 27.305))
+    (stroke (width 0) (type default) (color 0 0 0 0))
+  )
   (wire (pts (xy 33.02 88.265) (xy 21.59 88.265))
     (stroke (width 0) (type default) (color 0 0 0 0))
@@
     (stroke (width 0) (type default) (color 0 0 0 0))
   )
+  (wire (pts (xy 33.02 24.765) (xy 33.02 26.67))
+    (stroke (width 0) (type default) (color 0 0 0 0))
+  )
   (wire (pts (xy 66.04 36.195) (xy 62.865 36.195))
     (stroke (width 0) (type default) (color 0 0 0 0))
@@
     (stroke (width 0) (type default) (color 0 0 0 0))
   )
-  (wire (pts (xy 31.75 24.765) (xy 31.75 26.67))
-    (stroke (width 0) (type default) (color 0 0 0 0))
-  )
   (wire (pts (xy 21.59 84.455) (xy 21.59 85.725))
     (stroke (width 0) (type default) (color 0 0 0 0))
   )
+  (wire (pts (xy 159.385 57.785) (xy 168.275 57.785))
+    (stroke (width 0) (type default) (color 0 0 0 0))
+  )
   (wire (pts (xy 21.59 88.265) (xy 21.59 89.535))
     (stroke (width 0) (type default) (color 0 0 0 0))
@@
     (stroke (width 0) (type default) (color 0 0 0 0))
   )
-  (wire (pts (xy 31.75 34.29) (xy 31.75 36.195))
+  (wire (pts (xy 33.02 34.29) (xy 33.02 36.195))
     (stroke (width 0) (type default) (color 0 0 0 0))
   )
@@
     (stroke (width 0) (type default) (color 0 0 0 0))
   )
+  (wire (pts (xy 29.21 24.765) (xy 29.21 36.195))
+    (stroke (width 0) (type default) (color 0 0 0 0))
+  )
   (wire (pts (xy 41.275 24.765) (xy 41.275 26.67))
     (stroke (width 0) (type default) (color 0 0 0 0))
@@
     (stroke (width 0) (type default) (color 0 0 0 0))
   )
-  (wire (pts (xy 31.75 36.195) (xy 29.21 36.195))
+  (wire (pts (xy 33.02 36.195) (xy 29.21 36.195))
     (stroke (width 0) (type default) (color 0 0 0 0))
   )
@@
   (text "MCU\n" (at 155.575 18.415 0)
     (effects (font (size 2 2) (thickness 0.4) bold) (justify left bottom))
+  )
+  (text "pullup on D- to \nindicate USB low \nspeed device" (at 28.575 51.435 0)
+    (effects (font (size 1.27 1.27)) (justify left bottom))
   )
   (text "GPIO" (at 29.845 74.295 0)
@@
     (pin "8")
   )
-  (symbol (lib_id "power:+5V") (at 31.75 24.765 0) (unit 1)
-    (in_bom yes) (on_board yes) (fields_autoplaced)
-    (property "Reference" "#PWR0101" (id 0) (at 31.75 28.575 0)
-      (effects (font (size 1.27 1.27)) hide)
-    )
-    (property "Value" "+5V" (id 1) (at 31.75 19.685 0))
-    (property "Footprint" "" (id 2) (at 31.75 24.765 0)
-      (effects (font (size 1.27 1.27)) hide)
-    )
-    (property "Datasheet" "" (id 3) (at 31.75 24.765 0)
+  (symbol (lib_id "power:PWR_FLAG") (at 168.275 27.305 0) (unit 1)
+    (in_bom yes) (on_board yes) (fields_autoplaced)
+    (property "Reference" "#FLG0102" (id 0) (at 168.275 25.4 0)
+      (effects (font (size 1.27 1.27)) hide)
+    )
+    (property "Value" "PWR_FLAG" (id 1) (at 168.275 22.225 0))
+    (property "Footprint" "" (id 2) (at 168.275 27.305 0)
+      (effects (font (size 1.27 1.27)) hide)
+    )
+    (property "Datasheet" "~" (id 3) (at 168.275 27.305 0)
+      (effects (font (size 1.27 1.27)) hide)
+    )
+    (pin "1")
+  )
+  (symbol (lib_id "power:PWR_FLAG") (at 168.275 57.785 180) (unit 1)
+    (in_bom yes) (on_board yes) (fields_autoplaced)
+    (property "Reference" "#FLG0103" (id 0) (at 168.275 59.69 0)
+      (effects (font (size 1.27 1.27)) hide)
+    )
+    (property "Value" "PWR_FLAG" (id 1) (at 170.18 59.0549 0)
+      (effects (font (size 1.27 1.27)) (justify right))
+    )
+    (property "Footprint" "" (id 2) (at 168.275 57.785 0)
+      (effects (font (size 1.27 1.27)) hide)
+    )
+    (property "Datasheet" "~" (id 3) (at 168.275 57.785 0)
+      (effects (font (size 1.27 1.27)) hide)
+    )
+    (pin "1")
+  )
+  (symbol (lib_id "power:+5V") (at 33.02 24.765 0) (unit 1)
+    (in_bom yes) (on_board yes) (fields_autoplaced)
+    (property "Reference" "#PWR0101" (id 0) (at 33.02 28.575 0)
+      (effects (font (size 1.27 1.27)) hide)
+    )
+    (property "Value" "+5V" (id 1) (at 33.02 19.685 0))
+    (property "Footprint" "" (id 2) (at 33.02 24.765 0)
+      (effects (font (size 1.27 1.27)) hide)
+    )
+    (property "Datasheet" "" (id 3) (at 33.02 24.765 0)
       (effects (font (size 1.27 1.27)) hide)
     )
@@
       (effects (font (size 1.27 1.27)) (justify left))
     )
-    (property "Footprint" "Capacitor_THT:C_Disc_D6.0mm_W2.5mm_P5.00mm" (id 2) (at 112.0902 45.085 0)
+    (property "Footprint" "Capacitor_THT:CP_Radial_D4.0mm_P1.50mm" (id 2) (at 112.0902 45.085 0)
       (effects (font (size 1.27 1.27)) hide)
     )
@@
     )
     (property "Datasheet" "" (id 3) (at 21.59 53.975 0)
+      (effects (font (size 1.27 1.27)) hide)
+    )
+    (pin "1")
+  )
+  (symbol (lib_id "power:PWR_FLAG") (at 29.21 24.765 0) (unit 1)
+    (in_bom yes) (on_board yes)
+    (property "Reference" "#FLG0101" (id 0) (at 29.21 22.86 0)
+      (effects (font (size 1.27 1.27)) hide)
+    )
+    (property "Value" "PWR_FLAG" (id 1) (at 17.78 22.86 0)
+      (effects (font (size 1.27 1.27)) (justify left))
+    )
+    (property "Footprint" "" (id 2) (at 29.21 24.765 0)
+      (effects (font (size 1.27 1.27)) hide)
+    )
+    (property "Datasheet" "~" (id 3) (at 29.21 24.765 0)
       (effects (font (size 1.27 1.27)) hide)
     )
@@
     (pin "1")
   )
-  (symbol (lib_id "Device:D") (at 31.75 30.48 270) (unit 1)
-    (in_bom yes) (on_board yes) (fields_autoplaced)
-    (property "Reference" "D3" (id 0) (at 34.925 29.2099 90)
-      (effects (font (size 1.27 1.27)) (justify left))
-    )
-    (property "Value" "D" (id 1) (at 34.925 31.7499 90)
-      (effects (font (size 1.27 1.27)) (justify left))
-    )
-    (property "Footprint" "Diode_THT:D_A-405_P10.16mm_Horizontal" (id 2) (at 31.75 30.48 0)
-      (effects (font (size 1.27 1.27)) hide)
-    )
-    (property "Datasheet" "~" (id 3) (at 31.75 30.48 0)
+  (symbol (lib_id "Device:D") (at 33.02 30.48 270) (unit 1)
+    (in_bom yes) (on_board yes)
+    (property "Reference" "D3" (id 0) (at 34.925 29.21 90)
+      (effects (font (size 1.27 1.27)) (justify left))
+    )
+    (property "Value" "D" (id 1) (at 34.925 31.75 90)
+      (effects (font (size 1.27 1.27)) (justify left))
+    )
+    (property "Footprint" "Diode_THT:D_A-405_P10.16mm_Horizontal" (id 2) (at 33.02 30.48 0)
+      (effects (font (size 1.27 1.27)) hide)
+    )
+    (property "Datasheet" "~" (id 3) (at 33.02 30.48 0)
       (effects (font (size 1.27 1.27)) hide)
     )
@@
   )
   (symbol_instances
+    (path "/73fcdac2-d969-4b3d-ac11-2997b24fb4c4"
+      (reference "#FLG0101") (unit 1) (value "PWR_FLAG") (footprint "")
+    )
+    (path "/40cc65ce-d749-4210-8520-d1807a967eae"
+      (reference "#FLG0102") (unit 1) (value "PWR_FLAG") (footprint "")
+    )
+    (path "/4355055b-3fc3-4c72-80db-5db670324a86"
+      (reference "#FLG0103") (unit 1) (value "PWR_FLAG") (footprint "")
+    )
     (path "/4623f81a-3083-4b0b-81a8-66f51a010d1d"
       (reference "#PWR0101") (unit 1) (value "+5V") (footprint "")
@@
     )
     (path "/5a3519bf-2601-4320-9d02-484295fa808d"
-      (reference "C2") (unit 1) (value "4.7uF") (footprint "Capacitor_THT:C_Disc_D6.0mm_W2.5mm_P5.00mm")
+      (reference "C2") (unit 1) (value "4.7uF") (footprint "Capacitor_THT:CP_Radial_D4.0mm_P1.50mm")
     )
     (path "/826a0150-ddf3-4eec-861c-127f1472789a"

Commit message: Start new board and update QDev Tiny README
Other:
- title: QDevTiny ATtiny25/45/85 development board -> QDev Tiny ATtiny25/45/85 development board
